File: mawile/mawile.kicad_pcb (KiCad board)
At the start: 2 copper layers, 20 parts, among them J1 Conn_PiWR-Pi2C-PiLERTs, J2 Conn_A0x48-9, J3 Conn_A0x4A-B, U1 ADS1115, U2 ADS1115, U3 ADS1115, U4 ADS1115

Commit message: updated README
Parts:
- removed C3, C4, C5: 1uF, Capacitor_SMD:C_0805_2012Metric_Pad1.15x1.40mm_HandSolder
- removed FB1, FB2: MMZ2012Y152B, Inductor_SMD:L_0805_2012Metric_Pad1.15x1.40mm_HandSolder
- removed R1, R2, R3, R4, R5, R6: 10k, Resistor_SMD:R_0805_2012Metric_Pad1.15x1.40mm_HandSolder
- removed U1, U2, U3, U4: ADS1115, Radishes:VSSOP-10_2.4x2.1mm_P0.5mm
- added J4: I2C_O2, Connector_PinHeader_2.54mm:PinHeader_1x04_P2.54mm_Vertical, F.Cu at (87.1, 154.8)
- added J5: I2C_O3, Connector_PinHeader_2.54mm:PinHeader_1x04_P2.54mm_Vertical, F.Cu at (87.1, 157.4)
- C1: value 1uF -> 4.7uF; footprint Capacitor_THT:CP_Radial_D8.0mm_P3.80mm -> Capacitor_SMD:C_0805_2012Metric_Pad1.15x1.40mm_HandSolder; moved to B.Cu
- C2: value 1uF -> 4.7uF; moved to B.Cu
- J1: value Conn_PiWR-Pi2C-PiLERTs -> Pi/O_I2C; footprint Connector_Phoenix_MC_HighVoltage:PhoenixContact_MC_1,5_8-G-5.08_1x08_P5.08mm_Horizontal -> Connector_PinHeader_2.54mm:PinHeader_2x03_P2.54mm_Vertical
- J2: value Conn_A0x48-9 -> I2C_O0; footprint Connector_Phoenix_MC_HighVoltage:PhoenixContact_MC_1,5_8-G-5.08_1x08_P5.08mm_Horizontal -> Connector_PinHeader_2.54mm:PinHeader_1x04_P2.54mm_Vertical
- J3: value Conn_A0x4A-B -> I2C_O1; footprint Connector_Phoenix_MC_HighVoltage:PhoenixContact_MC_1,5_8-G-5.08_1x08_P5.08mm_Horizontal -> Connector_PinHeader_2.54mm:PinHeader_1x04_P2.54mm_Vertical
- moved C2 119.9 mm to (83.7, 151.1), turned to 90 degrees
- moved J2 73.8 mm to (87.1, 151.0), turned to 90 degrees
- moved J1 73.5 mm to (81.2, 154.8)
- moved C1 55.1 mm to (81.2, 151.1), turned to 90 degrees
- moved J3 42.7 mm to (87.1, 148.5), turned to 90 degrees
Connections:
- C1 pad 1: Net-(C1-Pad1) -> +3V3
- C1 pad 2: Net-(C1-Pad2) -> GNDD
- C2 pad 1: VDD -> +5V
- C2 pad 2: GND -> GNDD
- J1 pad 1: ALERT_0x4B -> +3V3
- J1 pad 2: ALERT_0x4A -> +5V
- J1 pad 3: ALERT_0x49 -> /SDA_Pi
- J1 pad 4: ALERT_0x48 -> +5V
- J1 pad 5: SDA -> /SCL_Pi
- J1 pad 6: Net-(C1-Pad2) -> GNDD
- J2 pad 1: Net-(J2-Pad1) -> +3V3
- J2 pad 2: Net-(J2-Pad2) -> /SDA_Pi
- J2 pad 3: Net-(J2-Pad3) -> /SCL_Pi
- J2 pad 4: Net-(J2-Pad4) -> GNDD
- J3 pad 1: Net-(J3-Pad1) -> +3V3
- J3 pad 2: Net-(J3-Pad2) -> /SDA_Pi
- J3 pad 3: Net-(J3-Pad3) -> /SCL_Pi
- J3 pad 4: Net-(J3-Pad4) -> GNDD
Routing:
- net /SCL_Pi: track 0.00 -> 44.8 mm
- net /SDA_Pi: track 0.00 -> 35.5 mm
- net +3V3: track 0.00 -> 14.2 mm
- net +5V: track 0.00 -> 2.54 mm
- net GNDD: vias 0 -> 4
- added copper zone on B.Cu, net +3V3
- added copper zone on F.Cu, net +5V
- added copper zone on B.Cu, net GNDD
- added copper zone on F.Cu, net GNDD
Other:
- net class Default: clearance 0.2 -> 0.1778
- rule trace_clearance: 0.2 -> 0.1778
- rule trace_min: 0.2 -> 0.127
- rule via_min_drill: 0.3 -> 0.254
- rule via_min_size: 0.4 -> 0.381
- board text added: "+3.3V"
- board text added: "+5V"
- board text added: "mawile"
- board text added: "mki ) 0 o ."
- board text added: "nubby, 2020"
