File: mawile/mawile.sch (KiCad schematic (older format))
At the start: 20 parts, among them J1 Conn_PiWR-Pi2C-PiLERTs, J2 Conn_A0x48-9, J3 Conn_A0x4A-B, U1 ADS1115, U2 ADS1115, U3 ADS1115, U4 ADS1115

Commit message: v2.0 schematic - outputs; may remove second buffer
Parts:
- removed C1: 1uF, Capacitor_THT:CP_Radial_D8.0mm_P3.80mm, symbol Device:CP1
- removed C2, C3, C4, C5: 1uF, Capacitor_SMD:C_0805_2012Metric_Pad1.15x1.40mm_HandSolder, symbol Device:C
- removed FB1, FB2: MMZ2012Y152B, Inductor_SMD:L_0805_2012Metric_Pad1.15x1.40mm_HandSolder, symbol Device:Ferrite_Bead
- removed J1: Conn_PiWR-Pi2C-PiLERTs, Connector_Phoenix_MC_HighVoltage:PhoenixContact_MC_1,5_8-G-5.08_1x08_P5.08mm_Horizontal, symbol Connector:Conn_01x08_Female
- removed J2: Conn_A0x48-9, Connector_Phoenix_MC_HighVoltage:PhoenixContact_MC_1,5_8-G-5.08_1x08_P5.08mm_Horizontal, symbol Connector:Conn_01x08_Female
- removed J3: Conn_A0x4A-B, Connector_Phoenix_MC_HighVoltage:PhoenixContact_MC_1,5_8-G-5.08_1x08_P5.08mm_Horizontal, symbol Connector:Conn_01x08_Female
- removed R1, R2, R3, R4, R5, R6: 10k, Resistor_SMD:R_0805_2012Metric_Pad1.15x1.40mm_HandSolder, symbol Device:R
- removed U1, U2, U3, U4: ADS1115, Radishes:VSSOP-10_2.4x2.1mm_P0.5mm, symbol radish:ADS1115
- added C? (x2): 4.7uF, symbol Device:C
- added C? (x4): 0.1uF, symbol Device:C_Small
- added J?: Pi/O_I2C, symbol Connector_Generic:Conn_02x03_Odd_Even
- added R? (x8): R, symbol Device:R
- added U? (x2): TCA9511A, symbol devs:TCA9511A
Connections:
- new net: C?.1, R?.2, U?.1 (ENABLE) (x2)
- new net: R?.2, U?.5 (READY) (x2)
- new net +3V3: C?.1, C?.1, C?.1, J?.1 (Pin_1), R?.1, R?.1, R?.1, R?.1, R?.1, R?.1, R?.1, R?.1, U?.7 (VDD), U?.7 (VDD)
- new net +5V: C?.1, J?.2 (Pin_2), J?.4 (Pin_4)
- new net GNDD: C?.2, C?.2, C?.2, C?.2, C?.2, C?.2, J?.6 (Pin_6), U?.4 (GND), U?.4 (GND)
- new net SCL_O1: R?.2, U?.2 (SCL_O), U?.3 (SCL_I)
- new net SCL_O2: U?.2 (SCL_O)
- new net SCL_Pi: J?.5 (Pin_5), R?.2, U?.3 (SCL_I)
- new net SDA_O1: R?.2, U?.6 (SDA_I), U?.7 (VDD)
- new net SDA_O2: U?.7 (VDD)
- new net SDA_Pi: J?.3 (Pin_3), R?.2, U?.6 (SDA_I)
Other:
- note added: "2.0"
- note added: "TODO :\n * Layout as shield for Pi.\n * Needs to accommodate soil sensor, temp/humidity sensors."
- note removed: "ADCs"
- note removed: "Address 0x48 (1001000)"
- note removed: "Address 0x49 (1001001)"
- note removed: "Address 0x4A (1001010)"
- note removed: "Address 0x4B (1001011)"
- note removed: "Pi/O"
- note removed: "TODO :\n * Layout\n * Needs to accommodate soil sensor, temp/humidity sensors."

Commit message: updated README
Parts:
- removed C? (x4): 0.1uF, symbol Device:C_Small
- removed R? (x8): R, symbol Device:R
- removed U? (x2): TCA9511A, symbol devs:TCA9511A
- added J2: I2C_O0, Connector_PinHeader_2.54mm:PinHeader_1x04_P2.54mm_Vertical, symbol Connector:Conn_01x04_Male
- added J3: I2C_O1, Connector_PinHeader_2.54mm:PinHeader_1x04_P2.54mm_Vertical, symbol Connector:Conn_01x04_Male
- added J4: I2C_O2, Connector_PinHeader_2.54mm:PinHeader_1x04_P2.54mm_Vertical, symbol Connector:Conn_01x04_Male
- added J5: I2C_O3, Connector_PinHeader_2.54mm:PinHeader_1x04_P2.54mm_Vertical, symbol Connector:Conn_01x04_Male
- C1, C2: renamed from C?; footprint (none) -> Capacitor_SMD:C_0805_2012Metric_Pad1.15x1.40mm_HandSolder
- J1: renamed from J?; footprint (none) -> Connector_PinHeader_2.54mm:PinHeader_2x03_P2.54mm_Vertical
Connections:
- net +3V3: now also J2.1 (Pin_1), J3.1 (Pin_1), J4.1 (Pin_1), J5.1 (Pin_1)
- net GNDD: now also J2.4 (Pin_4), J3.4 (Pin_4), J4.4 (Pin_4), J5.4 (Pin_4)
- net SCL_Pi: now also J2.3 (Pin_3), J3.3 (Pin_3), J4.3 (Pin_3), J5.3 (Pin_3)
- net SDA_Pi: now also J2.2 (Pin_2), J3.2 (Pin_2), J4.2 (Pin_2), J5.2 (Pin_2)
Other:
- moved on the sheet: C1, C2, J1
